File: dpedal.kicad_pcb (KiCad board)
At the start: 2 copper layers, 80 x 80 mm, 19 parts, among them J1 USB_C_Receptacle_USB2.0, SW1 SW_Push, SW2 SW_Push, SW3 SW_Push, SW4 SW_Push, SW5 RESET, SW6 FLASH, U1 STM32F072C8Tx, U2 LDO

Commit message: Getting ready to order
Parts:
- C7: value 100 nF -> 100nF
- moved SW2 9.27 mm to (90.0, 120.0), turned to 90 degrees
- moved SW1 8.99 mm to (60.0, 90.0), turned to 90 degrees
- moved SW4 6.04 mm to (120.0, 90.0), turned to 90 degrees
- moved C7 2.95 mm to (58.9, 103.1)
- moved SW3 1.21 mm to (90.0, 60.0), turned to 90 degrees
Connections:
- J1 pad A8: Net-(J1-PadA8) -> unconnected-(J1-PadA8)
- J1 pad B8: Net-(J1-PadA8) -> unconnected-(J1-PadB8)
Routing:
- net GND: track 50.9 -> 18.6 mm, vias 5 -> 1
- net Net-(SW1-Pad1): track 24.2 -> 32.0 mm
- net Net-(SW4-Pad2): track 38.6 -> 44.3 mm
- net Net-(C7-Pad2): track 25.4 -> 22.9 mm
- net Net-(SW2-Pad1): track 20.3 -> 18.9 mm
- net Net-(SW3-Pad2): track 44.9 -> 43.6 mm
- added copper zone on F.Cu, net GND
