File: dpedal.kicad_sch (KiCad schematic)
At the start: 3 parts

Commit message: progress
Parts:
- removed BT1: 3V, Battery:BatteryHolder_Keystone_1058_1x2032, symbol Device:Battery_Cell
- removed D1: red, LED_THT:LED_D5.0mm, symbol Device:LED
- added C1, C2: 1µF, Capacitor_SMD:C_0402_1005Metric, symbol Device:C
- added C3, C4, C5, C6: 100nF, Capacitor_SMD:C_0402_1005Metric, symbol Device:C
- added C7: 100 nF, Capacitor_SMD:C_0402_1005Metric, symbol Device:C
- added J1: USB_C_Receptacle_USB2.0, Connector_USB:USB_C_Receptacle_HRO_TYPE-C-31-M-12, symbol Connector:USB_C_Receptacle_USB2.0
- added R2, R3: 5.1K, Resistor_SMD:R_0402_1005Metric, symbol Device:R
- added SW1, SW2, SW3, SW4: SW_Push, Button_Switch_Keyboard:SW_Cherry_MX_1.00u_Plate, symbol Switch:SW_Push
- added SW5: RESET, Button_Switch_SMD:SW_SPST_CK_RS282G05A3, symbol Switch:SW_Push
- added SW6: FLASH, Button_Switch_SMD:SW_SPST_CK_RS282G05A3, symbol Switch:SW_Push
- added U1: STM32F072C8Tx, Package_QFP:LQFP-48_7x7mm_P0.5mm, symbol MCU_ST_STM32F0:STM32F072C8Tx
- added U2: LDO, Package_TO_SOT_SMD:SOT-23, symbol Regulator_Linear:MCP1703A-3302_SOT23
- R1: value 1K -> 5.1K; footprint Resistor_THT:R_Axial_DIN0309_L9.0mm_D3.2mm_P12.70mm_Horizontal -> Resistor_SMD:R_0402_1005Metric
Connections:
- net led is gone; now on net GND: R1.2
- net GND: now also C1.1, C2.1, C3.1, C4.1, C5.1, C6.1, C7.1, J1.A1 (GND), J1.A12 (GND), J1.B1 (GND), J1.B12 (GND), J1.S1 (SHIELD), R2.2, R3.2, SW1.2, SW2.2, SW3.1, SW4.1, SW5.1, U1.23 (VSS), U1.35 (VSS), U1.47 (VSS), U1.8 (VSSA), U2.1 (GND)
- net VCC: now also C1.2, J1.A4 (VBUS), J1.A9 (VBUS), J1.B4 (VBUS), J1.B9 (VBUS), U2.3 (VI); no longer R1.1
- new net: J1.A5 (CC1), R1.1
- new net: J1.A8 (SBU1), J1.B8 (SBU2)
- new net: J1.B5 (CC2), R2.1
- new net: SW4.2, U1.12 (PA2)
- new net: R3.1, SW6.2, U1.44 (BOOT0)
- new net: SW2.1, U1.11 (PA1)
- new net: SW3.2, U1.13 (PA3)
- new net: SW1.1, U1.14 (PA4)
- new net: C7.2, SW5.2, U1.7 (NRST)
- new net 3.3V: C2.2, C3.2, C4.2, C5.2, C6.2, SW6.1, U1.24 (VDD), U1.36 (VDDIO2), U1.48 (VDD), U1.9 (VDDA), U2.2 (VO)
- new net D+: J1.A6 (D+), J1.B6 (D+), U1.33 (PA12)
- new net D-: J1.A7 (D-), J1.B7 (D-), U1.32 (PA11)

Commit message: Getting ready to order
Parts:
- C7: value 100 nF -> 100nF
- J1: JLCPCB Part # (none) -> C165948
- SW1, SW2, SW3, SW4: now left out of the parts list
Connections:
- net at J1.A8 (SBU1): no longer J1.B8 (SBU2)
Changed lines of the file:
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@@
-    (stroke (width 0) (type default) (color 0 0 0 0))
-  )
-  (wire (pts (xy 45.72 64.77) (xy 45.72 67.31))
     (stroke (width 0) (type default) (color 0 0 0 0))
   )
@@
     )
     (property "Datasheet" "https://www.usb.org/sites/default/files/documents/usb_type-c.zip" (id 3) (at 34.29 52.07 0)
+      (effects (font (size 1.27 1.27)) hide)
+    )
+    (property "JLCPCB Part #" "C165948" (id 4) (at 30.48 52.07 0)
       (effects (font (size 1.27 1.27)) hide)
     )
@@
   )
   (symbol (lib_id "Switch:SW_Push") (at 180.34 96.52 180) (unit 1)
-    (in_bom yes) (on_board yes) (fields_autoplaced)
+    (in_bom no) (on_board yes) (fields_autoplaced)
     (property "Reference" "SW4" (id 0) (at 180.34 91.44 0))
     (property "Value" "SW_Push" (id 1) (at 180.34 93.98 0))
@@
     (pin "2")
   )
-  (symbol (lib_id "power:PWR_FLAG") (at 49.53 36.83 0) (unit 1)
+  (symbol (lib_name "PWR_FLAG_1") (lib_id "power:PWR_FLAG") (at 49.53 36.83 0) (unit 1)
     (in_bom yes) (on_board yes)
     (property "Reference" "#FLG0102" (id 0) (at 49.53 34.925 0)
@@
     (pin "1")
   )
-  (symbol (lib_id "power:GND") (at 106.68 82.55 0) (unit 1)
+  (symbol (lib_name "GND_5") (lib_id "power:GND") (at 106.68 82.55 0) (unit 1)
     (in_bom yes) (on_board yes)
     (property "Reference" "#PWR03" (id 0) (at 106.68 88.9 0)
@@
     (pin "1")
   )
-  (symbol (lib_id "power:GND") (at 185.42 101.6 90) (unit 1)
+  (symbol (lib_name "GND_1") (lib_id "power:GND") (at 185.42 101.6 90) (unit 1)
     (in_bom yes) (on_board yes) (fields_autoplaced)
     (property "Reference" "#PWR0102" (id 0) (at 191.77 101.6 0)
@@
     (pin "2")
   )
-  (symbol (lib_id "power:GND") (at 57.15 43.18 90) (unit 1)
+  (symbol (lib_name "GND_6") (lib_id "power:GND") (at 57.15 43.18 90) (unit 1)
     (in_bom yes) (on_board yes) (fields_autoplaced)
     (property "Reference" "#PWR0101" (id 0) (at 63.5 43.18 0)
@@
     (pin "2")
   )
-  (symbol (lib_id "power:GND") (at 137.16 41.91 180) (unit 1)
+  (symbol (lib_name "GND_2") (lib_id "power:GND") (at 137.16 41.91 180) (unit 1)
     (in_bom yes) (on_board yes) (fields_autoplaced)
     (property "Reference" "#PWR0103" (id 0) (at 137.16 35.56 0)
@@
     (pin "2")
   )
-  (symbol (lib_id "power:GND") (at 78.74 44.45 0) (unit 1)
+  (symbol (lib_name "GND_3") (lib_id "power:GND") (at 78.74 44.45 0) (unit 1)
     (in_bom yes) (on_board yes) (fields_autoplaced)
     (property "Reference" "#PWR0104" (id 0) (at 78.74 50.8 0)
@@
       (effects (font (size 1.27 1.27)) hide)
     )
-    (pin "1")
-    (pin "2")
-  )
-  (symbol (lib_id "power:GND") (at 36.83 74.93 0) (unit 1)
+    (property "Field4" "" (id 4) (at 100.33 73.66 0)
+      (effects (font (size 1.27 1.27)) hide)
+    )
+    (pin "1")
+    (pin "2")
+  )
+  (symbol (lib_name "GND_7") (lib_id "power:GND") (at 36.83 74.93 0) (unit 1)
     (in_bom yes) (on_board yes) (fields_autoplaced)
     (property "Reference" "#PWR02" (id 0) (at 36.83 81.28 0)
@@
       (effects (font (size 1.27 1.27)) (justify left))
     )
-    (property "Value" "100 nF" (id 1) (at 97.79 60.96 0)
+    (property "Value" "100nF" (id 1) (at 97.79 60.96 0)
       (effects (font (size 1.27 1.27)) (justify left))
     )
@@
   )
   (symbol (lib_id "Switch:SW_Push") (at 180.34 118.11 0) (unit 1)
-    (in_bom yes) (on_board yes) (fields_autoplaced)
+    (in_bom no) (on_board yes) (fields_autoplaced)
     (property "Reference" "SW1" (id 0) (at 180.34 110.49 0))
     (property "Value" "SW_Push" (id 1) (at 180.34 113.03 0))
@@
   )
   (symbol (lib_id "Switch:SW_Push") (at 180.34 106.68 180) (unit 1)
-    (in_bom yes) (on_board yes) (fields_autoplaced)
+    (in_bom no) (on_board yes) (fields_autoplaced)
     (property "Reference" "SW3" (id 0) (at 180.34 101.6 0))
     (property "Value" "SW_Push" (id 1) (at 180.34 104.14 0))
@@
     (pin "2")
   )
-  (symbol (lib_id "power:GND") (at 102.87 54.61 180) (unit 1)
+  (symbol (lib_name "GND_4") (lib_id "power:GND") (at 102.87 54.61 180) (unit 1)
     (in_bom yes) (on_board yes) (fields_autoplaced)
     (property "Reference" "#PWR0105" (id 0) (at 102.87 48.26 0)
@@
   )
   (symbol (lib_id "Switch:SW_Push") (at 180.34 86.36 0) (unit 1)
-    (in_bom yes) (on_board yes) (fields_autoplaced)
+    (in_bom no) (on_board yes) (fields_autoplaced)
     (property "Reference" "SW2" (id 0) (at 180.34 78.74 0))
     (property "Value" "SW_Push" (id 1) (at 180.34 81.28 0))
@@
     )
     (path "/c02217c5-d179-4e4a-8419-33cf676fa2be"
-      (reference "C7") (unit 1) (value "100 nF") (footprint "Capacitor_SMD:C_0402_1005Metric")
+      (reference "C7") (unit 1) (value "100nF") (footprint "Capacitor_SMD:C_0402_1005Metric")
     )
     (path "/05a051cd-5697-4628-9a41-57143ebaa4a5"

Commit message: Ordered design
Parts:
- C1, C2: LCSC C282732 -> C52923
- R1, R2, R3: JLCPCB Part # (none) -> C25905
- SW5, SW6: JLCPCB Part # (none) -> C5117870
- U1: JLCPCB Part # (none) -> C80488; JLCPCB Rotation Offset (none) -> 270
- U2: JLCPCB Rotation Offset (none) -> 180
Changed lines of the file:
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@@
+      (effects (font (size 1.27 1.27)) hide)
+    )
+    (property "JLCPCB Part #" "C25905" (id 4) (at 106.68 77.47 0)
       (effects (font (size 1.27 1.27)) hide)
     )
@@
     )
     (property "Datasheet" "http://www.st.com/st-web-ui/static/active/en/resource/technical/document/datasheet/DM00090510.pdf" (id 3) (at 132.08 97.79 0)
+      (effects (font (size 1.27 1.27)) hide)
+    )
+    (property "JLCPCB Part #" "C80488" (id 4) (at 132.08 97.79 0)
+      (effects (font (size 1.27 1.27)) hide)
+    )
+    (property "JLCPCB Rotation Offset" "270" (id 5) (at 132.08 97.79 0)
       (effects (font (size 1.27 1.27)) hide)
     )
@@
       (effects (font (size 1.27 1.27)) hide)
     )
+    (property "JLCPCB Part #" "C5117870" (id 4) (at 106.68 59.69 90)
+      (effects (font (size 1.27 1.27)) hide)
+    )
     (pin "1")
     (pin "2")
@@
       (effects (font (size 1.27 1.27)) hide)
     )
+    (property "JLCPCB Part #" "C25905" (id 4) (at 53.34 40.64 90)
+      (effects (font (size 1.27 1.27)) hide)
+    )
     (pin "1")
     (pin "2")
@@
       (effects (font (size 1.27 1.27)) hide)
     )
-    (property "LCSC" "C282732" (id 4) (at 107.95 45.72 0)
+    (property "LCSC" "C52923" (id 4) (at 107.95 45.72 0)
       (effects (font (size 1.27 1.27)) hide)
     )
@@
       (effects (font (size 1.27 1.27)) hide)
     )
-    (property "Field4" "" (id 4) (at 100.33 73.66 0)
+    (property "JLCPCB Part #" "C5117870" (id 4) (at 100.33 73.66 0)
       (effects (font (size 1.27 1.27)) hide)
     )
@@
       (effects (font (size 1.27 1.27)) hide)
     )
+    (property "JLCPCB Rotation Offset" "180" (id 5) (at 83.82 36.83 0)
+      (effects (font (size 1.27 1.27)) hide)
+    )
     (pin "1")
     (pin "2")
@@
       (effects (font (size 1.27 1.27)) hide)
     )
+    (property "JLCPCB Part #" "C25905" (id 4) (at 53.34 45.72 90)
+      (effects (font (size 1.27 1.27)) hide)
+    )
     (pin "1")
     (pin "2")
@@
       (effects (font (size 1.27 1.27)) hide)
     )
-    (property "LCSC" "C282732" (id 4) (at 73.66 40.64 0)
-      (effects (font (size 1.27 1.27)) hide)
-    )
+    (property "LCSC" "C52923" (id 4) (at 73.66 40.64 0)
+      (effects (font (size 1.27 1.27)) hide)
+    )
