File: PCB/dpedal.kicad_pcb (KiCad board)
At the start: 2 copper layers, 80 x 80 mm, 19 parts, among them J1 USB_C_Receptacle_USB2.0, SW1 SW_Push, SW2 SW_Push, SW3 SW_Push, SW4 SW_Push, SW5 RESET, SW6 FLASH, U1 STM32F072C8Tx, U2 LDO

Commit message: PCB v2
Parts:
- added J2: Conn_02x10_Counter_Clockwise, Connector_IDC:IDC-Header_2x10_P2.54mm_Horizontal, F.Cu at (134.0, 116.0)
- added J3: Conn_ARM_JTAG_SWD_10, Connector_PinHeader_1.27mm:PinHeader_2x05_P1.27mm_Vertical, F.Cu at (43.0, 107.0)
- added SW10: SW_Push, Switch_Keyboard_Hotswap_Kailh:SW_Hotswap_Kailh_MX_plated_1.00u, F.Cu at (157.0, 60.0)
- added SW7: SW_Push, Switch_Keyboard_Hotswap_Kailh:SW_Hotswap_Kailh_MX_plated_1.00u, F.Cu at (23.0, 120.0)
- added SW8: SW_Push, Switch_Keyboard_Hotswap_Kailh:SW_Hotswap_Kailh_MX_plated_1.00u, F.Cu at (157.0, 120.0)
- added SW9: SW_Push, Switch_Keyboard_Hotswap_Kailh:SW_Hotswap_Kailh_MX_plated_1.00u, F.Cu at (23.0, 60.0)
- SW1, SW2, SW3, SW4: footprint Button_Switch_Keyboard:SW_Cherry_MX_1.00u_Plate -> Switch_Keyboard_Hotswap_Kailh:SW_Hotswap_Kailh_MX_plated_1.00u
Connections:
- U1 pad 15: unconnected-(U1-Pad15) -> Net-(SW7-Pad1)
- U1 pad 16: unconnected-(U1-Pad16) -> Net-(SW8-Pad1)
- U1 pad 17: unconnected-(U1-Pad17) -> Net-(SW9-Pad1)
- U1 pad 18: unconnected-(U1-Pad18) -> Net-(J2-Pad1)
- U1 pad 19: unconnected-(U1-Pad19) -> Net-(J2-Pad2)
- U1 pad 20: unconnected-(U1-Pad20) -> Net-(J2-Pad3)
- U1 pad 21: unconnected-(U1-Pad21) -> Net-(J2-Pad11)
- U1 pad 22: unconnected-(U1-Pad22) -> Net-(J2-Pad12)
- U1 pad 25: unconnected-(U1-Pad25) -> Net-(J2-Pad13)
- U1 pad 26: unconnected-(U1-Pad26) -> Net-(J2-Pad14)
- U1 pad 27: unconnected-(U1-Pad27) -> Net-(J2-Pad15)
- U1 pad 28: unconnected-(U1-Pad28) -> Net-(J2-Pad16)
- U1 pad 29: unconnected-(U1-Pad29) -> Net-(SW10-Pad1)
- U1 pad 30: unconnected-(U1-Pad30) -> Net-(J2-Pad19)
- U1 pad 31: unconnected-(U1-Pad31) -> Net-(J2-Pad18)
- U1 pad 34: unconnected-(U1-Pad34) -> SWDIO
- U1 pad 37: unconnected-(U1-Pad37) -> SWDCLK
- U1 pad 38: unconnected-(U1-Pad38) -> Net-(J2-Pad17)
- U1 pad 39: unconnected-(U1-Pad39) -> Net-(J2-Pad4)
- U1 pad 40: unconnected-(U1-Pad40) -> Net-(J2-Pad5)
- U1 pad 41: unconnected-(U1-Pad41) -> Net-(J2-Pad6)
- U1 pad 42: unconnected-(U1-Pad42) -> Net-(J2-Pad7)
- U1 pad 43: unconnected-(U1-Pad43) -> Net-(J2-Pad8)
- U1 pad 45: unconnected-(U1-Pad45) -> Net-(J2-Pad9)
- U1 pad 46: unconnected-(U1-Pad46) -> Net-(J2-Pad10)
Routing:
- net GND: track 18.6 -> 157.5 mm
- net Net-(SW4-Pad2): track 44.3 -> 0.00 mm
- net Net-(SW3-Pad2): track 43.6 -> 0.00 mm
- net Net-(SW1-Pad1): track 32.0 -> 0.00 mm
- net Net-(SW2-Pad1): track 18.9 -> 0.00 mm
Other:
- board size 80 x 80 mm -> 154 x 80 mm
- board text added: "DPedal V2"
- board text removed: "DPedal V1"

Commit message: PCB v2 More
Parts:
- added J4: Conn_01x05, Connector_PinHeader_1.00mm:PinHeader_1x05_P1.00mm_Horizontal, F.Cu at (64.0, 53.8)
- moved J3 3.16 mm to (46.0, 108.0)
- moved C2 2.51 mm to (76.0, 115.1)
- moved C1 1.97 mm to (76.6, 120.1)
- moved U2 1.97 mm to (76.0, 117.6)
- moved R2 1.36 mm to (68.6, 119.0)
- moved R1 1.15 mm to (68.5, 120.0)
- moved C5 1.00 mm to (77.0, 112.8)
- moved C7 1.00 mm to (58.9, 102.1), turned to -90 degrees
- moved C3 0.43 mm to (67.3, 110.2)
- moved C6 0.24 mm to (70.0, 101.2)
- moved C4 0.18 mm to (78.8, 106.0)
Connections:
- J2 pad 1: Net-(J2-Pad1) -> GND
- J2 pad 10: Net-(J2-Pad10) -> EXT10
- J2 pad 11: Net-(J2-Pad11) -> EXT11
- J2 pad 12: Net-(J2-Pad12) -> EXT12
- J2 pad 13: Net-(J2-Pad13) -> EXT13
- J2 pad 14: Net-(J2-Pad14) -> EXT14
- J2 pad 15: Net-(J2-Pad15) -> EXT15
- J2 pad 16: Net-(J2-Pad16) -> EXT16
- J2 pad 17: Net-(J2-Pad17) -> EXT17
- J2 pad 18: Net-(J2-Pad18) -> EXT18
- J2 pad 19: Net-(J2-Pad19) -> EXT19
- J2 pad 2: Net-(J2-Pad2) -> EXT2
- J2 pad 20: GND -> EXT20
- J2 pad 3: Net-(J2-Pad3) -> EXT3
- J2 pad 4: Net-(J2-Pad4) -> EXT4
- J2 pad 5: Net-(J2-Pad5) -> EXT5
- J2 pad 6: Net-(J2-Pad6) -> EXT6
- J2 pad 7: Net-(J2-Pad7) -> EXT7
- J2 pad 8: Net-(J2-Pad8) -> EXT8
- J2 pad 9: Net-(J2-Pad9) -> EXT9
- SW1 pad 1: Net-(SW1-Pad1) -> SW1
- SW10 pad 1: Net-(SW10-Pad1) -> SW10
- SW2 pad 1: Net-(SW2-Pad1) -> SW2
- SW3 pad 2: Net-(SW3-Pad2) -> SW3
- SW4 pad 2: Net-(SW4-Pad2) -> SW4
- SW7 pad 1: Net-(SW7-Pad1) -> SW7
- SW8 pad 1: Net-(SW8-Pad1) -> GND
- SW8 pad 2: GND -> SW8
- SW9 pad 1: Net-(SW9-Pad1) -> SW9
- U1 pad 10: unconnected-(U1-Pad10) -> EXT6
- U1 pad 11: Net-(SW2-Pad1) -> EXT8
- U1 pad 12: Net-(SW4-Pad2) -> EXT10
- U1 pad 13: Net-(SW3-Pad2) -> EXT12
- U1 pad 14: Net-(SW1-Pad1) -> EXT14
- U1 pad 15: Net-(SW7-Pad1) -> EXT16
- U1 pad 16: Net-(SW8-Pad1) -> EXT18
- U1 pad 17: Net-(SW9-Pad1) -> EXT20
- U1 pad 18: Net-(J2-Pad1) -> EXT19
- U1 pad 19: Net-(J2-Pad2) -> EXT17
- U1 pad 2: unconnected-(U1-Pad2) -> SW2
- U1 pad 20: Net-(J2-Pad3) -> EXT15
- U1 pad 21: Net-(J2-Pad11) -> EXT13
- U1 pad 22: Net-(J2-Pad12) -> EXT11
- U1 pad 25: Net-(J2-Pad13) -> SW1
- U1 pad 26: Net-(J2-Pad14) -> EXT9
- U1 pad 27: Net-(J2-Pad15) -> EXT7
- U1 pad 28: Net-(J2-Pad16) -> EXT5
- U1 pad 29: Net-(SW10-Pad1) -> EXT3
- U1 pad 3: unconnected-(U1-Pad3) -> EXT2
- U1 pad 30: Net-(J2-Pad19) -> SW4
- U1 pad 31: Net-(J2-Pad18) -> SW8
- U1 pad 38: Net-(J2-Pad17) -> SW10
- U1 pad 39: Net-(J2-Pad4) -> SW3
- U1 pad 4: unconnected-(U1-Pad4) -> EXT4
- U1 pad 40: Net-(J2-Pad5) -> PEDAL4
- U1 pad 41: Net-(J2-Pad6) -> PEDAL3
- U1 pad 42: Net-(J2-Pad7) -> PEDAL2
- U1 pad 43: Net-(J2-Pad8) -> PEDAL1
- U1 pad 45: Net-(J2-Pad9) -> SW9
- U1 pad 46: Net-(J2-Pad10) -> SW7
Routing:
- net SW8: track 0.00 -> 219.8 mm, vias 0 -> 1
- net SW10: track 0.00 -> 189.3 mm, vias 0 -> 1
- net EXT3: track 0.00 -> 159.5 mm
- net EXT5: track 0.00 -> 155.3 mm
- net EXT7: track 0.00 -> 151.0 mm
- net EXT9: track 0.00 -> 146.9 mm
- net GND: track 157.5 -> 24.5 mm, vias 1 -> 7
- net SW3: track 0.00 -> 127.4 mm, vias 0 -> 1
- net SW4: track 0.00 -> 121.3 mm, vias 0 -> 1
- net PEDAL1: track 0.00 -> 116.6 mm
- net PEDAL2: track 0.00 -> 115.3 mm
- net PEDAL3: track 0.00 -> 114.0 mm
- net PEDAL4: track 0.00 -> 112.8 mm
- net SW9: track 0.00 -> 96.9 mm, vias 0 -> 1
- net EXT2: track 0.00 -> 68.1 mm
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