File: PCB/dpedal.kicad_pcb (KiCad board)
At the start: 2 copper layers, 154 x 80 mm, 26 parts, among them J1 USB_C_Receptacle_USB2.0, J2 Conn_02x10_Counter_Clockwise, J3 Conn_ARM_JTAG_SWD_10, J4 Conn_01x05, SW1 SW_Push, SW10 SW_Push, SW2 SW_Push, SW3 SW_Push, SW4 SW_Push, SW5 RESET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

Commit message: Update symbols/footprints
Parts:
- U2: footprint Package_TO_SOT_SMD:SOT-23 -> Package_TO_SOT_SMD:SOT-23-3
- moved C1 0.21 mm to (76.5, 120.2)
Connections:
- U1 pad 1: unconnected-(U1-Pad1) -> 3.3V
Routing:
- net GND: track 24.5 -> 23.9 mm
