File: pcb/dpedal_pcb.kicad_pcb (KiCad board)
At the start: 2 copper layers, 126.5 x 55.5 mm, 7 parts, among them SW1 SW_Push, SW2 SW_Push, SW3 SW_Push, SW4 SW_Push, SW5 SW_Push, SW6 SW_Push

Commit message: tweak pcb
Connections:
- A1 pad 17: unconnected-(A1-GPIO13-Pad17) -> button_left
- A1 pad 19: button_left -> unconnected-(A1-GPIO14-Pad19)
Routing:
- net GND: track 2.96 -> 0.00 mm, vias 4 -> 5
- net button_left: track 13.3 -> 12.4 mm
Changed lines of the file:
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@@
 	(net 23 "unconnected-(A1-GPIO10-Pad14)")
 	(net 24 "unconnected-(A1-GPIO12-Pad16)")
-	(net 25 "unconnected-(A1-GPIO13-Pad17)")
+	(net 25 "unconnected-(A1-GPIO14-Pad19)")
 	(net 26 "unconnected-(A1-GPIO6-Pad9)")
 	(net 27 "GND")
@@
 		)
 		(fp_text user "${REFERENCE}"
-			(at -3.69 -19 90)
+			(at -3.69 -19 180)
 			(layer "B.Fab")
 			(effects
@@
 			(layers "B.Cu" "B.Mask")
 			(roundrect_rratio 0.5)
-			(net 25 "unconnected-(A1-GPIO13-Pad17)")
+			(net 5 "button_left")
 			(pinfunction "GPIO13")
-			(pintype "bidirectional+no_connect")
+			(pintype "bidirectional")
 		)
 		(pad "18" smd custom
@@
 			(layers "B.Cu" "B.Mask")
 			(roundrect_rratio 0.5)
-			(net 5 "button_left")
+			(net 25 "unconnected-(A1-GPIO14-Pad19)")
 			(pinfunction "GPIO14")
-			(pintype "bidirectional")
+			(pintype "bidirectional+no_connect")
 		)
 		(pad "20" smd roundrect
@@
 			(pinfunction "GND")
 			(pintype "passive")
+			(thermal_bridge_angle 90)
 			(options
 				(clearance outline)
@@
 	)
 	(segment
-		(start 105.15 140.15)
-		(end 109.59 144.59)
+		(start 114.96 139.51)
+		(end 104.64 139.51)
 		(width 0.2)
 		(layer "B.Cu")
@@
 	)
 	(segment
-		(start 104 140.15)
-		(end 105.15 140.15)
+		(start 104.64 139.51)
+		(end 104 140.15)
 		(width 0.2)
 		(layer "B.Cu")
@@
 	)
 	(segment
-		(start 109.59 144.59)
-		(end 115.46 144.59)
+		(start 104 140.15)
+		(end 105.15 140.15)
 		(width 0.2)
 		(layer "B.Cu")
@@
 	)
 	(segment
-		(start 143.564093 133.15)
-		(end 149 133.15)
+		(start 139.5 136.5)
+		(end 142.85 133.15)
 		(width 0.2)
 		(layer "B.Cu")
@@
 	)
 	(segment
-		(start 139.5 137.214093)
-		(end 143.564093 133.15)
+		(start 139.5 142)
+		(end 139.5 136.5)
 		(width 0.2)
 		(layer "B.Cu")
@@
 	)
 	(segment
-		(start 139.5 142)
-		(end 139.5 137.214093)
+		(start 136.91 144.59)
+		(end 139.5 142)
 		(width 0.2)
 		(layer "B.Cu")
@@
 	)
 	(segment
-		(start 136.91 144.59)
-		(end 139.5 142)
+		(start 142.85 133.15)
+		(end 149 133.15)
 		(width 0.2)
 		(layer "B.Cu")
@@
 	)
 	(via
+		(at 143 145)
+		(size 0.6)
+		(drill 0.3)
+		(layers "F.Cu" "B.Cu")
+		(free yes)
+		(net 27)
+	)
+	(via
 		(at 143.5 114.5)
 		(size 0.6)
@@
 		(net 27)
 	)
-	(segment
-		(start 125.15 144.15)
-		(end 125 144)
-		(width 0.2)
-		(layer "B.Cu")
-		(net 27)
-	)
-	(segment
-		(start 125.15 146.9)
-		(end 125.15 144.15)
-		(width 0.2)
-		(layer "B.Cu")
-		(net 27)
-	)

Commit message: silkscreen
Connections:
- SW4 pad 1: dpad_left -> GND
- SW4 pad 2: GND -> dpad_left
Routing:
- net dpad_left: track 22.1 -> 13.8 mm
Other:
- board text added: "DPedal V3"
- board text added: "by rukai"
