File: pcb/dpedal_pcb.kicad_pcb (KiCad board)
At the start: 2 copper layers, 126.5 x 55.5 mm, 7 parts, among them SW1 SW_Push, SW2 SW_Push, SW3 SW_Push, SW4 SW_Push, SW5 SW_Push, SW6 SW_Push

Commit message: Add website address to PCB silkscreen
Other:
- board text added: "To build and configure:"
- board text added: "dpedal.com"
Changed lines of the file:
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@@
+		)
+	)
+	(gr_text "To build and configure:"
+		(at 203.085712 148.5 -0)
+		(layer "B.SilkS")
+		(effects
+			(font
+				(size 2 2)
+				(thickness 0.5)
+			)
+			(justify mirror)
+		)
+	)
+	(gr_text "dpedal.com"
+		(at 204 154 0)
+		(layer "B.SilkS")
+		(effects
+			(font
+				(size 4 4)
+				(thickness 0.9)
+				(bold yes)
+			)
+			(justify mirror)
 		)
 	)
